File: LoRa-Dev.kicad_pcb (KiCad board)
At the start: 4 copper layers, 56 x 71 mm, 19 parts, among them J1 Conn_Coaxial_Small, J2 Barrel_Jack_MountingPin, U1 RPi Pico, U2 LT1963AEQ, U5 RFM95W-868S2

Commit message: RFM95PW wrong branch name
Parts:
- removed J1: Conn_Coaxial_Small, Connector_Coaxial:U.FL_Hirose_U.FL-R-SMT-1_Vertical
- removed U5: RFM95W-868S2, LoRa-Dev:RFM95W
- added J3: Conn_Coaxial_Small, Connector_Coaxial:U.FL_Hirose_U.FL-R-SMT-1_Vertical, F.Cu at (100.3, 61.7)
- added U3: RFM95PW, LoRa-Dev:RFM95PW, F.Cu at (111.0, 77.8)
- R7: value 2K2 -> 4k7
- R8: value 1K2 -> 1K5
- moved R9 33.4 mm to (93.5, 49.6), turned to 90 degrees
- moved C3 3.28 mm to (124.7, 65.5)
- moved C4 2.50 mm to (124.0, 59.0)
Connections:
- U1 pad 26: (no net) -> /DIO0
Routing:
- net /DIO0: track 0.00 -> 52.3 mm, vias 0 -> 4
- net RF_VDD: track 70.6 -> 109.1 mm, vias 4 -> 6
- net /SPI_SCK: track 70.0 -> 36.2 mm
- net /RESETn: track 57.7 -> 25.4 mm, vias 1 -> 0
- net /SPI_MOSI: track 57.0 -> 36.4 mm
- net /SPI_MISO: track 60.7 -> 43.1 mm
- net /DIO1: track 46.5 -> 54.5 mm, vias 1 -> 4
- net /SPI_CSn: track 54.6 -> 47.3 mm, vias 1 -> 3
- net /ANT: track 15.3 -> 11.1 mm
- net GND: vias 35 -> 50
- net /RF_GND: vias 0 -> 29
Other:
- board size 56 x 71 mm -> 72.5 x 71 mm

Commit message: fixed
Parts:
- moved R9 1.75 mm to (93.5, 47.8)
- moved U3 0.75 mm to (111.8, 77.8)
Routing:
- net /RESETn: track 25.4 -> 26.0 mm
Changed lines of the file:
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@@
 	(footprint "LoRa-Dev:RFM95PW"
 		(layer "F.Cu")
-		(at 111.0325 77.75 180)
+		(at 111.7825 77.75 180)
 		(property "Reference" "U3"
-			(at 1.016 -2.667 360)
+			(at 1.016 -2.667 0)
 			(layer "F.SilkS")
 			(hide yes)
@@
 		)
 		(property "Value" "RFM95PW"
-			(at -4.318 7.6835 360)
+			(at -4.318 7.6835 0)
 			(layer "F.SilkS")
 			(hide yes)
@@
 		)
 		(property "Footprint" "LoRa-Dev:RFM95PW"
-			(at 0 0 360)
+			(at 0 0 0)
 			(layer "F.Fab")
 			(hide yes)
@@
 		)
 		(property "Datasheet" ""
-			(at 0 0 360)
+			(at 0 0 0)
 			(layer "F.Fab")
 			(hide yes)
@@
 		)
 		(property "Description" ""
-			(at 0 0 360)
+			(at 0 0 0)
 			(layer "F.Fab")
 			(hide yes)
@@
 		)
 		(fp_text user "RADIO 2"
-			(at 5.08 -6.1595 360)
+			(at 5.08 -6.1595 0)
 			(layer "F.SilkS")
 			(hide yes)
@@
 			(at 0 -1.43 0)
 			(layer "F.SilkS")
+			(hide yes)
 			(effects
 				(font
@@
 	(footprint "Resistor_SMD:R_0603_1608Metric"
 		(layer "F.Cu")
-		(at 93.5 49.575 90)
+		(at 93.5 47.825 90)
 		(descr "Resistor SMD 0603 (1608 Metric), square (rectangular) end terminal, IPC_7351 nominal, (Body size source: IPC-SM-782 page 72, https://www.pcb-3d.com/wordpress/wp-content/uploads/ipc-sm-782a_amendment_1_and_2.pdf), generated with kicad-footprint-generator")
 		(tags "resistor")
@@
 	)
 	(via
+		(at 95 47)
+		(size 0.6)
+		(drill 0.3)
+		(layers "F.Cu" "B.Cu")
+		(free yes)
+		(net 2)
+	)
+	(via
 		(at 152.5 63.5)
 		(size 0.6)
@@
 	)
 	(via
-		(at 93.5 47.25)
+		(at 93.5 45.75)
 		(size 0.6)
 		(drill 0.3)
@@
 	)
 	(via
-		(at 109.25 76.25)
+		(at 109.25 77.5)
 		(size 0.6)
 		(drill 0.3)
@@
 	)
 	(via
-		(at 92 47.25)
+		(at 92 45.75)
 		(size 0.6)
 		(drill 0.3)
@@
 	)
 	(via
-		(at 138.5 62.5)
-		(size 0.6)
-		(drill 0.3)
-		(layers "F.Cu" "B.Cu")
-		(net 2)
-	)
-	(via
-		(at 125.75 55)
+		(at 92 47)
 		(size 0.6)
 		(drill 0.3)
@@
 	)
 	(via
-		(at 126.75 68.75)
+		(at 138.5 62.5)
 		(size 0.6)
 		(drill 0.3)
 		(layers "F.Cu" "B.Cu")
-		(free yes)
 		(net 2)
 	)
 	(via
-		(at 133.5 62.5)
+		(at 125.75 55)
 		(size 0.6)
 		(drill 0.3)
 		(layers "F.Cu" "B.Cu")
+		(free yes)
 		(net 2)
 	)
 	(via
-		(at 126.75 70.75)
+		(at 126.75 68.75)
 		(size 0.6)
 		(drill 0.3)
@@
 	)
 	(via
-		(at 100.5 78)
+		(at 133.5 62.5)
 		(size 0.6)
 		(drill 0.3)
 		(layers "F.Cu" "B.Cu")
-		(free yes)
 		(net 2)
 	)
 	(via
-		(at 95 48.75)
+		(at 126.75 70.75)
 		(size 0.6)
 		(drill 0.3)
@@
 	)
 	(via
-		(at 92 48.75)
+		(at 100.5 78)
 		(size 0.6)
 		(drill 0.3)
@@
 	)
 	(via
-		(at 109.25 78)
+		(at 110.75 80)
 		(size 0.6)
 		(drill 0.3)
@@
 	)
 	(via
-		(at 95 47.25)
+		(at 95 45.75)
 		(size 0.6)
 		(drill 0.3)
@@
 	)
 	(segment
-		(start 128.7825 74.25)
-		(end 130.69 72.3425)
+		(start 130.69 73.31)
+		(end 130.69 50)
 		(width 0.254)
 		(layer "F.Cu")
@@
 	)
 	(segment
-		(start 130.69 72.3425)
-		(end 130.69 50)
+		(start 129.75 74.25)
+		(end 130.69 73.31)
 		(width 0.254)
 		(layer "F.Cu")
@@
 	(segment
 		(start 128.4325 74.25)
-		(end 128.7825 74.25)
+		(end 129.75 74.25)
 		(width 0.254)
 		(layer "F.Cu")
@@
 	)
 	(zone
-		(net 2)
-		(net_name "GND")
-		(layer "F.Cu")
-		(hatch edge 0.5)
-		(priority 9)
-		(connect_pads yes
-			(clearance 0.253)
-		)
-		(min_thickness 0.253)
-		(filled_areas_thickness no)
-		(fill yes
-			(thermal_gap 0.5)
-			(thermal_bridge_width 0.5)
-		)
-		(polygon
-			(pts
-				(xy 90.5 29) (xy 128 29) (xy 128 49.5) (xy 90.5 49.5)
-			)
-		)
-	)
-	(zone
 		(net 1)
 		(net_name "Net-(U2-IN)")
@@
 		(polygon
 			(pts
-				(xy 90.5 48.5) (xy 122.75 48.5) (xy 122.75 71.25) (xy 90.5 71.25)
+				(xy 90.5 48.25) (xy 122.75 48.25) (xy 122.75 71) (xy 90.5 71)
 			)
 		)
@@
 		(polygon
 			(pts
-				(xy 123.25 29) (xy 123.25 71.25) (xy 90.5 71.25) (xy 90.5 100) (xy 163 100) (xy 163 29)
+				(xy 123.25 29) (xy 90.5 29) (xy 90.75 49.5) (xy 123.5 49.5) (xy 123.25 49.75) (xy 123.25 71.5) (xy 90.5 71.5)
+				(xy 90.5 100) (xy 163 100) (xy 163 29)
 			)
 		)
@@
 		(polygon
 			(pts
-				(xy 95.75 68.25) (xy 127 68.25) (xy 127 86.25) (xy 95.75 86.25)
+				(xy 102.5 78.75) (xy 109 78.75) (xy 109 85.75) (xy 102.5 85.75)
+			)
+		)
+	)
+	(zone
+		(net 0)
+		(net_name "")
+		(layer "F.SilkS")
+		(hatch edge 0.5)
+		(priority 4)
+		(connect_pads yes
+			(clearance 0.253)
+		)
+		(min_thickness 0.253)
+		(filled_areas_thickness no)
+		(fill yes
+			(thermal_gap 0.5)
+			(thermal_bridge_width 0.5)
+		)
+		(polygon
+			(pts
+				(xy 102.5 68.75) (xy 109 68.75) (xy 109 72.5) (xy 102.5 72.5)
+			)
+		)
+	)
+	(zone
+		(net 0)
+		(net_name "")
+		(layer "F.SilkS")
+		(hatch edge 0.5)
+		(priority 4)
+		(connect_pads yes
+			(clearance 0.253)
+		)
+		(min_thickness 0.253)
+		(filled_areas_thickness no)
+		(fill yes
+			(thermal_gap 0.5)
+			(thermal_bridge_width 0.5)
+		)
+		(polygon
+			(pts
+				(xy 95.25 68.75) (xy 102.25 68.75) (xy 102.25 85.75) (xy 95.25 85.75)
+			)
+		)
+	)
+	(zone
+		(net 0)
+		(net_name "")
+		(layer "F.SilkS")
+		(hatch edge 0.5)
+		(priority 4)
+		(connect_pads yes
+			(clearance 0.253)
+		)
+		(min_thickness 0.253)
+		(filled_areas_thickness no)
+		(fill yes
+			(thermal_gap 0.5)
+			(thermal_bridge_width 0.5)
+		)
+		(polygon
+			(pts
+				(xy 109.25 68.75) (xy 127.75 68.75) (xy 127.75 85.75) (xy 109.25 85.75)
 			)
 		)

Commit message: updated after first review
Parts:
- removed C4: 47uF, Capacitor_SMD:CP_Elec_6.3x5.8
- added C5: 47uf, Capacitor_SMD:C_1210_3225Metric, F.Cu at (125.0, 59.2)
- moved J3 1.41 mm to (101.2, 60.7)
- moved C3 0.25 mm to (125.0, 65.5)
Connections:
- U1 pad 20: unconnected-(U1-GP15-Pad20) -> /DIO5
- U1 pad 31: unconnected-(U1-GP26-Pad31) -> /DIO2
- U1 pad 32: unconnected-(U1-GP27-Pad32) -> /DIO3
- U1 pad 34: unconnected-(U1-GP28-Pad34) -> /DIO4
- U3 pad 15: unconnected-(U3-DIO5-Pad15) -> /DIO5
- U3 pad 2: GND -> /RF_GND
- U3 pad 3: unconnected-(U3-DIO3-Pad3) -> /DIO3
- U3 pad 4: unconnected-(U3-DIO4-Pad4) -> /DIO4
- U3 pad 8: unconnected-(U3-DIO2-Pad8) -> /DIO2
Routing:
- net /DIO2: track 0.00 -> 90.4 mm, vias 0 -> 2
- net /DIO3: track 0.00 -> 89.4 mm, vias 0 -> 2
- net /DIO4: track 0.00 -> 88.8 mm, vias 0 -> 2
- net /DIO5: track 0.00 -> 50.4 mm, vias 0 -> 2
- net RF_VDD: track 109.1 -> 91.8 mm, vias 6 -> 5
- net /SPI_CSn: track 47.3 -> 52.6 mm
- net /RESETn: track 26.0 -> 28.9 mm, vias 0 -> 1
- net /SPI_SCK: track 36.2 -> 33.6 mm
- net /SPI_MOSI: track 36.4 -> 34.2 mm
- net /ANT: track 11.1 -> 12.3 mm
- net GND: vias 50 -> 46
